Commit message: initial ACHD solver setup and control

File: openarm_compl_ctrl/urdf/openarm_bimanual.urdf (robot description, URDF)
Before this commit: robot openarm, 26 links, 25 joints
Links:
- link openarm_left_link7: mass 0.4659771327380578 -> 0.8880281327380577
- link openarm_right_link7: mass 0.4659771327380578 -> 0.8880281327380577

Commit message: fix motor comm, add msg for pid debug, update plotter

File: openarm_compl_ctrl/urdf/openarm_bimanual.urdf (robot description, URDF)
Before this commit: robot openarm, 26 links, 25 joints
Links:
- link openarm_left_link7: mass 0.8880281327380577 -> 0.4659771327380578

Commit message: refractor robot comm into a library

File: openarm_compl_ctrl/urdf/openarm_bimanual.urdf (robot description, URDF)
Before this commit: robot openarm, 26 links, 25 joints
Joints:
- joint openarm_left_finger_joint1: type prismatic -> fixed
- joint openarm_left_finger_joint2: type prismatic -> fixed
- joint openarm_right_finger_joint1: type prismatic -> fixed
- joint openarm_right_finger_joint2: type prismatic -> fixed

Commit message: updates

File: openarm_compl_ctrl/urdf/openarm_bimanual.urdf (robot description, URDF)
Before this commit: robot openarm, 26 links, 25 joints
Links:
- link openarm_right_link7: mass 0.8880281327380577 -> 0.4659771327380578
